Commit message: Add 3-camera Nav2 costmap integration for autonomous navigation
This commit implements the complete integration of 3 ZED2i cameras with
RTAB-Map SLAM and Nav2 costmaps for the Exodus rover's autonomous
navigation system.

Changes:
- Update RTAB-Map config for 3 cameras with grid map publishing
  * Enable Grid/FromDepth for 2D occupancy grid generation
  * Configure all 3 camera serials (32514439, 31718458, 33289078)
  * Add point cloud publishing at 15Hz

- Create Nav2 costmap configuration (costmap_params.yaml)
  * Global costmap: subscribes to /rtabmap/grid_map
  * Local costmap: uses voxel layer with 3 camera point clouds
  * Proper inflation layers for safety margins

- Add costmap launch file (costmap_bringup.launch.py)
  * Launches global and local costmap nodes
  * Remaps /map to /rtabmap/grid_map for RTAB-Map integration
  * Includes lifecycle manager for Nav2 activation

- Update camera URDF for 3rd camera
  * Add camera3 (manipulator mount) at (0.2, 0.0, 1.2)
  * 30° downward tilt for manipulation tasks
  * Complete 360° coverage with all 3 cameras

- Add comprehensive documentation
  * NAVIGATION_SETUP.md: System architecture and troubleshooting
  * JETSON_DEPLOYMENT.md: Jetson deployment and testing guide

This resolves the issue where RTAB-Map and costmap were disconnected
in rqt_graph. The costmap now properly receives SLAM data for
autonomous navigation.

🤖 Generated with [Claude Code](https://claude.com/claude-code)

Co-Authored-By: Claude Sonnet 4.5 <noreply@anthropic.com>

File: mobility_ctrl/src/nav2_stanley/urdf/zed_cameras.xacro.urdf (robot description, URDF)
Before this commit: robot zed_cameras, 0 links, 2 joints
Joints:
- added joint $(arg camera_name_3)_joint: type fixed, parent base_link, child $(arg camera_name_3)_camera_link, origin xyz=0.2 0.0 1.2 rpy=0 0.524 0
